File: REF1395A Optimized.kicad_pcb (KiCad board)
At the start: 2 copper layers, 83.5 x 129.8 mm, 21 parts, among them J1 Cart_Edge_Connector, J2 Game_Edge_Connector, J3 SW_DPDT_x2, J4 Conn_01x16_Male, J5 Conn_01x16_Male, J6 Conn_01x20_Male, J7 Conn_01x20_Male, J8 Conn_01x20_Male, J9 Conn_01x20_Male, Q1 BC847C, SW1 SW_Push_Dual, U1 SST39SF010, U2 V62C5181024L-70W, U3 GBASICV3 ORBIT 61676

Commit message: Add files via upload
Other:
- board text added: "GND Rail"
Changed lines of the file:
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@@
+    (effects (font (size 1 1) (thickness 0.15)))
+  )
+  (gr_text "GND Rail" (at 114.52 101.228) (layer "F.SilkS")
     (effects (font (size 1 1) (thickness 0.15)))
   )
@@
     (effects (font (size 1 1) (thickness 0.15)))
   )
+  (gr_text "GND Rail" (at 174.718 101.228) (layer "F.SilkS")
+    (effects (font (size 1 1) (thickness 0.15)))
+  )
   (gr_text "10K Ohm" (at 180.469 79.658 270) (layer "F.SilkS")
     (effects (font (size 0.5 0.5) (thickness 0.125)))
+  )
+  (gr_text "GND Rail" (at 174.718 114.931) (layer "F.SilkS")
+    (effects (font (size 1 1) (thickness 0.15)))
   )
   (gr_text "100 nF" (at 159.539 174.475) (layer "F.SilkS")
@@
     (effects (font (size 1 1) (thickness 0.15)))
   )
+  (gr_text "GND Rail" (at 114.52 114.931) (layer "F.SilkS")
+    (effects (font (size 1 1) (thickness 0.15)))
+  )
+  (gr_text "GND Rail" (at 169.871 128.947) (layer "F.SilkS")
+    (effects (font (size 1 1) (thickness 0.15)))
+  )
+  (gr_text "GND Rail" (at 119.707 128.947) (layer "F.SilkS")
+    (effects (font (size 1 1) (thickness 0.15)))
+  )
